Commit message: Before first trial

File: description/gazebo_control.xacro (robot description, xacro)
@@ -2,5 +2,8 @@
 <robot xmlns:xacro="http://www.ros.org/wiki/xacro">
     <gazebo>
-        <plugin name='diff_drive' filename='libgazebo_ros_diff_drive.so'>
+        <plugin filename="libgazebo_ros2_control.so" name="gazebo_ros2_control">
+            <!-- <parameters>
+                $(find pico_bot)/config/my_controllers.yaml
+            </parameters> -->
             <!-- Wheel Information -->
             <left_joint>left_wheel_joint</left_joint>
@@ -10,5 +13,5 @@
             <!-- Limits -->
             <max_wheel_torque>100</max_wheel_torque>
-            <max_wheel_acceleration>2</max_wheel_acceleration>
+            <max_wheel_acceleration>10</max_wheel_acceleration>
             <!-- Output -->
             <odometry_frame>odom</odometry_frame>

File: description/robot.urdf.xacro (robot description, xacro)
@@ -1,7 +1,13 @@
 <?xml version="1.0"?>
 <robot xmlns:xacro="http://www.ros.org/wiki/xacro"  name="robot">
+    <xacro:arg name="use_ros2_control" default="true"/>
+    <xacro:if value="$(arg use_ros2_control)">
+        <xacro:include filename="ros2_control.xacro" />
+    </xacro:if>
+    <xacro:unless value="$(arg use_ros2_control)">
+        <xacro:include filename="gazebo_control.xacro" />
+    </xacro:unless>
     <xacro:include filename="robot_core.xacro"/>
     <xacro:include filename="inertial_macros.xacro"/>
-    <xacro:include filename="gazebo_control.xacro"/>
     <xacro:include filename="lidar.xacro"/>
 </robot>

File: description/robot_core.xacro (robot description, xacro)
@@ -7,4 +7,5 @@
         <parent link="base_link"/>
         <child link="chassis"/>
+        <!-- <origin xyz="0 0 0" rpy="0 0 0"/> -->
     </joint>
     <link name="chassis">
@@ -54,5 +55,5 @@
         <collision>
             <geometry>
-                <cylinder length="0.035" radius="0.04" />
+                <sphere radius="0.04" />
             </geometry>
         </collision>
@@ -81,5 +82,5 @@
         <collision>
             <geometry>
-                <cylinder length="0.035" radius="0.04" />
+                <sphere radius="0.04" />
             </geometry>
         </collision>
@@ -96,5 +97,5 @@
     </joint>
     <link name="caster_wheel">
-        <xacro:inertial_sphere mass="0.1" radius="0.04">
+        <xacro:inertial_sphere mass="0.5" radius="0.04"> <!-- Mass changed to 0.5 to fix tilting,, previous mass was 0.1-->
             <origin xyz="0 0 0" rpy="0 0 0"/>
         </xacro:inertial_sphere>

Commit message: Before ROS2 control real

File: description/gazebo_control.xacro (robot description, xacro)
@@ -12,6 +12,6 @@
             <wheel_diameter>0.08</wheel_diameter>
             <!-- Limits -->
-            <max_wheel_torque>100</max_wheel_torque>
-            <max_wheel_acceleration>10</max_wheel_acceleration>
+            <max_wheel_torque>200</max_wheel_torque>
+            <max_wheel_acceleration>10.0</max_wheel_acceleration>
             <!-- Output -->
             <odometry_frame>odom</odometry_frame>

File: description/robot.urdf.xacro (robot description, xacro)
@@ -1,4 +1,6 @@
 <?xml version="1.0"?>
 <robot xmlns:xacro="http://www.ros.org/wiki/xacro"  name="robot">
+    <!-- deleted xacro including of inertial_macros.xacro-->
+    <xacro:include filename="robot_core.xacro"/>
     <xacro:arg name="use_ros2_control" default="true"/>
     <xacro:if value="$(arg use_ros2_control)">
@@ -8,6 +10,4 @@
         <xacro:include filename="gazebo_control.xacro" />
     </xacro:unless>
-    <xacro:include filename="robot_core.xacro"/>
-    <xacro:include filename="inertial_macros.xacro"/>
     <xacro:include filename="lidar.xacro"/>
 </robot>

File: description/robot_core.xacro (robot description, xacro)
@@ -7,5 +7,5 @@
         <parent link="base_link"/>
         <child link="chassis"/>
-        <!-- <origin xyz="0 0 0" rpy="0 0 0"/> -->
+        <origin xyz="0 0 0" rpy="0 0 0"/>
     </joint>
     <link name="chassis">
@@ -49,5 +49,5 @@
         <visual>
             <geometry>
-                <cylinder length="0.035" radius="0.04" />
+                <cylinder length="0.035" radius="0.04"/>
             </geometry>
             <material name="blue"/>
@@ -55,5 +55,5 @@
         <collision>
             <geometry>
-                <sphere radius="0.04" />
+                <cylinder length="0.035" radius="0.04"/>
             </geometry>
         </collision>
@@ -82,5 +82,5 @@
         <collision>
             <geometry>
-                <sphere radius="0.04" />
+                <cylinder length="0.035" radius="0.04"/>
             </geometry>
         </collision>

File: description/ros2_control.xacro (robot description, xacro)
@@ -18,11 +18,10 @@
                 <param name="max">10</param>
             </command_interface>
+            <state_interface name="position" />
             <state_interface name="velocity" />
-            <state_interface name="position" />
         </joint>
     </ros2_control>
     <gazebo>
         <plugin filename="libgazebo_ros2_control.so" name="gazebo_ros2_control">
-            <robot_sim_type>gazebo_ros2_control/GazeboSystem</robot_sim_type>
             <parameters>$(find pico_bot)/config/my_controllers.yaml</parameters>
         </plugin>
